File: eagle/Board_1_controller_v1.brd (EAGLE design)
At the start: 14 x 57 mm, 29 parts, among them U3 ATMEGA328, Y1 8Mhz

Commit message: Latest Update, research files added
Parts:
- R1, R4: value 330 -> 47
- R5: value 330 -> 85
- R7, R8: value 330 -> 150
Connections:
- net BUTT1: now also U3.16
Routing:
- net BUTT1: track 5.36 -> 9.22 mm
Changed lines of the file:
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@@
 <attribute name="VALUE" x="9.516" y="46.0795" size="0.4064" layer="27" rot="R180"/>
 </element>
-<element name="R1" library="SparkFun" package="0402-RES" value="330" x="3.75" y="34" smashed="yes" rot="R270">
+<element name="R1" library="SparkFun" package="0402-RES" value="47" x="3.75" y="34" smashed="yes" rot="R270">
 <attribute name="NAME" x="3.4485" y="36.789" size="0.6" layer="25" rot="R270"/>
 </element>
-<element name="R4" library="SparkFun" package="0402-RES" value="330" x="5" y="34" smashed="yes" rot="R270">
+<element name="R4" library="SparkFun" package="0402-RES" value="47" x="5" y="34" smashed="yes" rot="R270">
 <attribute name="NAME" x="4.6985" y="36.789" size="0.6" layer="25" rot="R270"/>
 </element>
-<element name="R5" library="SparkFun" package="0402-RES" value="330" x="10.75" y="34" smashed="yes" rot="R270">
+<element name="R5" library="SparkFun" package="0402-RES" value="85" x="10.75" y="34" smashed="yes" rot="R270">
 <attribute name="NAME" x="10.4485" y="36.889" size="0.6" layer="25" rot="R270"/>
 </element>
@@
 <attribute name="NAME" x="11.5985" y="36.889" size="0.6" layer="25" rot="R270"/>
 </element>
-<element name="R7" library="SparkFun" package="0402-RES" value="330" x="2.25" y="34" smashed="yes" rot="R270">
+<element name="R7" library="SparkFun" package="0402-RES" value="150" x="2.25" y="34" smashed="yes" rot="R270">
 <attribute name="NAME" x="1.9485" y="36.889" size="0.6" layer="25" rot="R270"/>
 </element>
-<element name="R8" library="SparkFun" package="0402-RES" value="330" x="1" y="34" smashed="yes" rot="R270">
+<element name="R8" library="SparkFun" package="0402-RES" value="150" x="1" y="34" smashed="yes" rot="R270">
 <attribute name="NAME" x="0.7985" y="36.889" size="0.6" layer="25" rot="R270"/>
 </element>
@@
 <via x="7" y="23.8" extent="1-16" drill="0.4318"/>
 <wire x1="7" y1="23.8" x2="7" y2="20.65" width="0.4064" layer="16"/>
+<contactref element="U3" pad="16"/>
+<wire x1="8.055425" y1="21.515225" x2="8.8" y2="22.2598" width="0.4064" layer="1"/>
+<wire x1="8.8" y1="22.2598" x2="8.8" y2="22.9" width="0.4064" layer="1"/>
+<wire x1="8.8" y1="22.9" x2="7.9" y2="23.8" width="0.4064" layer="1"/>
+<wire x1="7.9" y1="23.8" x2="7" y2="23.8" width="0.4064" layer="1"/>
 </signal>
 <signal name="GRN">
