File: eagle/Board_1_controller_v1.sch (EAGLE design)
At the start: 29 parts, among them U3 ATMEGA328, Y1 8Mhz

Commit message: Latest Update, research files added
Parts:
- R1, R4: value 330 -> 47
- R5: value 330 -> 85
- R7, R8: value 330 -> 150
Connections:
- net BUTT1: now also U3.PB4(MISO)
Changed lines of the file:
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@@
 <part name="GRN1" library="IdleHandsProject" deviceset="LED" device="0603"/>
 <part name="GRN2" library="IdleHandsProject" deviceset="LED" device="0603"/>
-<part name="R1" library="SparkFun" deviceset="RESISTOR" device="0402-RES" value="330"/>
-<part name="R4" library="SparkFun" deviceset="RESISTOR" device="0402-RES" value="330"/>
-<part name="R5" library="SparkFun" deviceset="RESISTOR" device="0402-RES" value="330"/>
+<part name="R1" library="SparkFun" deviceset="RESISTOR" device="0402-RES" value="47"/>
+<part name="R4" library="SparkFun" deviceset="RESISTOR" device="0402-RES" value="47"/>
+<part name="R5" library="SparkFun" deviceset="RESISTOR" device="0402-RES" value="85"/>
 <part name="R6" library="SparkFun" deviceset="RESISTOR" device="0402-RES" value="330"/>
-<part name="R7" library="SparkFun" deviceset="RESISTOR" device="0402-RES" value="330"/>
-<part name="R8" library="SparkFun" deviceset="RESISTOR" device="0402-RES" value="330"/>
+<part name="R7" library="SparkFun" deviceset="RESISTOR" device="0402-RES" value="150"/>
+<part name="R8" library="SparkFun" deviceset="RESISTOR" device="0402-RES" value="150"/>
 <part name="SG1" library="SparkFun-Electromechanical" deviceset="BUZZER" device="PTH"/>
 <part name="GND2" library="SparkFun" deviceset="GND" device=""/>
@@
 <label x="195.58" y="43.18" size="1.778" layer="95"/>
 </segment>
-</net>
+<segment>
+<pinref part="U3" gate="G$1" pin="PB4(MISO)"/>
+<wire x1="175.26" y1="10.16" x2="187.96" y2="10.16" width="0.1524" layer="91"/>
+<label x="180.34" y="10.16" size="1.778" layer="95"/>
+</segment>
+</net>
