File: eagle/Board_2_sensor_v1.sch (EAGLE design)
At the start: 20 parts, among them CN2 M02JST-PTH-2, IC7 TLV71333DBV, U1 MCP3421, U2 MCP73831, X1 Micro USB

Commit message: Latest Update, research files added
Parts:
- removed L1: (no value), SparkFun-Passives:INDUCTOR0402
- added RP2: 22k, SparkFun:RESISTOR0402-RES
- added RP3: 180k, SparkFun:RESISTOR0402-RES
- added U$3: OPA344, SparkFun-AnalogIC:OPA344
Connections:
- removed net N$1: C2.2, L1.2, U1.VDD
- removed net N$5: LED1.C, RP1.2, U1.VIN+
- new net N$2: LED1.A, RP1.2, U$3.+IN
- new net N$3: RP2.1, RP3.1, U$3.-IN
- new net N$4: RP3.2, U$3.OUT, U1.VIN+
- net GND: now also C2.2, LED1.C, RP2.2, U$3.V-; no longer LED1.A
- net VCC: now also U$3.V+, U1.VDD; no longer L1.1
Other:
- moved on the sheet: LED1, RP1
Changed lines of the file:
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@@
 <part name="LED1" library="IdleHandsProject" deviceset="MTPD1346" device=""/>
 <part name="U1" library="IdleHandsProject" deviceset="MCP3421" device=""/>
-<part name="GND3" library="SparkFun" deviceset="GND" device=""/>
 <part name="GND4" library="SparkFun" deviceset="GND" device=""/>
 <part name="C7" library="rcl" deviceset="C-EU" device="C0402" value="0.1uF"/>
@@
 <part name="RP1" library="SparkFun" deviceset="RESISTOR" device="0402-RES" value="1M"/>
 <part name="JP2" library="SparkFun-Connectors" deviceset="M06" device="SMD-1MM"/>
-<part name="L1" library="SparkFun-Passives" deviceset="INDUCTOR" device="0402"/>
 <part name="SUPPLY1" library="SparkFun-Aesthetics" deviceset="3.3V" device=""/>
 <part name="C2" library="SparkFun" deviceset="CAP" device="0402-CAP" value="0.1uF"/>
@@
 <part name="SUPPLY2" library="SparkFun-Aesthetics" deviceset="3.3V" device=""/>
 <part name="SUPPLY3" library="SparkFun-Aesthetics" deviceset="3.3V" device=""/>
+<part name="U$3" library="SparkFun-AnalogIC" deviceset="OPA344" device=""/>
+<part name="RP2" library="SparkFun" deviceset="RESISTOR" device="0402-RES" value="22k"/>
+<part name="RP3" library="SparkFun" deviceset="RESISTOR" device="0402-RES" value="180k"/>
+<part name="P+1" library="SparkFun" deviceset="VCC" device="" value="3.3V"/>
+<part name="GND3" library="SparkFun" deviceset="GND" device=""/>
 </parts>
 <sheets>
@@
 <instance part="C1" gate="G$1" x="81.28" y="22.86"/>
 <instance part="X1" gate="G$1" x="12.7" y="27.94" rot="MR0"/>
-<instance part="LED1" gate="G$1" x="63.5" y="81.28" rot="R270"/>
+<instance part="LED1" gate="G$1" x="45.72" y="78.74" rot="R180"/>
 <instance part="U1" gate="G$1" x="119.38" y="78.74"/>
-<instance part="GND3" gate="1" x="66.04" y="63.5"/>
 <instance part="GND4" gate="1" x="119.38" y="53.34"/>
 <instance part="C7" gate="G$1" x="127" y="15.24"/>
@@
 <instance part="P+6" gate="1" x="160.02" y="27.94"/>
 <instance part="S1" gate="1" x="114.3" y="30.48"/>
-<instance part="P+2" gate="1" x="83.82" y="111.76"/>
+<instance part="P+2" gate="1" x="45.72" y="119.38"/>
 <instance part="GND6" gate="1" x="91.44" y="55.88"/>
-<instance part="GND8" gate="1" x="73.66" y="66.04"/>
-<instance part="RP1" gate="G$1" x="83.82" y="99.06" rot="R270"/>
+<instance part="GND8" gate="1" x="45.72" y="63.5"/>
+<instance part="RP1" gate="G$1" x="45.72" y="109.22" rot="R270"/>
 <instance part="JP2" gate="G$1" x="228.6" y="48.26" rot="R180"/>
-<instance part="L1" gate="G$1" x="119.38" y="106.68"/>
 <instance part="SUPPLY1" gate="G$1" x="119.38" y="121.92"/>
 <instance part="C2" gate="G$1" x="132.08" y="104.14"/>
@@
 <instance part="SUPPLY2" gate="G$1" x="152.4" y="104.14"/>
 <instance part="SUPPLY3" gate="G$1" x="167.64" y="93.98"/>
+<instance part="U$3" gate="G$1" x="63.5" y="96.52"/>
+<instance part="RP2" gate="G$1" x="55.88" y="78.74" rot="R270"/>
+<instance part="RP3" gate="G$1" x="78.74" y="111.76"/>
+<instance part="P+1" gate="1" x="63.5" y="119.38"/>
+<instance part="GND3" gate="1" x="132.08" y="93.98"/>
 </instances>
 <busses>
@@
 </segment>
 <segment>
-<pinref part="GND3" gate="1" pin="GND"/>
-<wire x1="66.04" y1="66.04" x2="66.04" y2="71.12" width="0.1524" layer="91"/>
-<wire x1="66.04" y1="71.12" x2="64.77" y2="71.12" width="0.1524" layer="91"/>
-<pinref part="LED1" gate="G$1" pin="CASE"/>
-<wire x1="64.77" y1="71.12" x2="63.5" y2="71.12" width="0.1524" layer="91"/>
-<junction x="64.77" y="71.12"/>
-</segment>
-<segment>
 <wire x1="91.44" y1="73.66" x2="91.44" y2="58.42" width="0.1524" layer="91"/>
 <pinref part="GND6" gate="1" pin="GND"/>
 <pinref part="U1" gate="G$1" pin="VIN-"/>
 <wire x1="91.44" y1="73.66" x2="104.14" y2="73.66" width="0.1524" layer="91"/>
-</segment>
-<segment>
-<pinref part="LED1" gate="G$1" pin="A"/>
-<wire x1="68.58" y1="81.28" x2="73.66" y2="81.28" width="0.1524" layer="91"/>
-<wire x1="73.66" y1="81.28" x2="73.66" y2="68.58" width="0.1524" layer="91"/>
-<pinref part="GND8" gate="1" pin="GND"/>
+<junction x="91.44" y="73.66"/>
+<pinref part="RP2" gate="G$1" pin="2"/>
+<wire x1="55.88" y1="73.66" x2="63.5" y2="73.66" width="0.1524" layer="91"/>
+<pinref part="U$3" gate="G$1" pin="V-"/>
+<wire x1="63.5" y1="73.66" x2="91.44" y2="73.66" width="0.1524" layer="91"/>
+<wire x1="63.5" y1="88.9" x2="63.5" y2="73.66" width="0.1524" layer="91"/>
+<junction x="63.5" y="73.66"/>
 </segment>
 <segment>
@@
 <wire x1="223.52" y1="40.64" x2="213.36" y2="40.64" width="0.1524" layer="91"/>
 <label x="213.36" y="40.64" size="1.778" layer="95"/>
+</segment>
+<segment>
+<pinref part="LED1" gate="G$1" pin="C"/>
+<wire x1="35.56" y1="73.66" x2="45.72" y2="73.66" width="0.1524" layer="91"/>
+<pinref part="GND8" gate="1" pin="GND"/>
+<wire x1="45.72" y1="73.66" x2="45.72" y2="66.04" width="0.1524" layer="91"/>
+<junction x="45.72" y="73.66"/>
+<wire x1="35.56" y1="78.74" x2="35.56" y2="77.47" width="0.1524" layer="91"/>
+<pinref part="LED1" gate="G$1" pin="CASE"/>
+<wire x1="35.56" y1="77.47" x2="35.56" y2="73.66" width="0.1524" layer="91"/>
+<junction x="35.56" y="77.47"/>
+</segment>
+<segment>
+<pinref part="C2" gate="G$1" pin="2"/>
+<wire x1="132.08" y1="101.6" x2="132.08" y2="96.52" width="0.1524" layer="91"/>
+<pinref part="GND3" gate="1" pin="GND"/>
 </segment>
 </net>
@@
 <segment>
 <pinref part="P+2" gate="1" pin="VCC"/>
-<wire x1="83.82" y1="104.14" x2="83.82" y2="111.76" width="0.1524" layer="91"/>
+<wire x1="45.72" y1="114.3" x2="45.72" y2="119.38" width="0.1524" layer="91"/>
 <pinref part="RP1" gate="G$1" pin="1"/>
 </segment>
@@
 <segment>
 <pinref part="SUPPLY1" gate="G$1" pin="3.3V"/>
-<pinref part="L1" gate="G$1" pin="1"/>
 <wire x1="119.38" y1="121.92" x2="119.38" y2="116.84" width="0.1524" layer="91"/>
 <pinref part="C2" gate="G$1" pin="1"/>
-<wire x1="119.38" y1="116.84" x2="119.38" y2="114.3" width="0.1524" layer="91"/>
 <wire x1="119.38" y1="116.84" x2="132.08" y2="116.84" width="0.1524" layer="91"/>
 <wire x1="132.08" y1="116.84" x2="132.08" y2="109.22" width="0.1524" layer="91"/>
+<pinref part="U1" gate="G$1" pin="VDD"/>
+<wire x1="119.38" y1="91.44" x2="119.38" y2="116.84" width="0.1524" layer="91"/>
 <junction x="119.38" y="116.84"/>
 </segment>
@@
 <pinref part="R4" gate="G$1" pin="1"/>
 <wire x1="167.64" y1="93.98" x2="167.64" y2="88.9" width="0.1524" layer="91"/>
+</segment>
+<segment>
+<pinref part="U$3" gate="G$1" pin="V+"/>
+<pinref part="P+1" gate="1" pin="VCC"/>
+<wire x1="63.5" y1="104.14" x2="63.5" y2="119.38" width="0.1524" layer="91"/>
 </segment>
 </net>
@@
 </segment>
 </net>
-<net name="N$5" class="0">
-<segment>
-<pinref part="LED1" gate="G$1" pin="C"/>
-<wire x1="60.96" y1="81.28" x2="60.96" y2="88.9" width="0.1524" layer="91"/>
-<wire x1="60.96" y1="88.9" x2="83.82" y2="88.9" width="0.1524" layer="91"/>
+<net name="N$2" class="0">
+<segment>
+<pinref part="RP1" gate="G$1" pin="2"/>
+<pinref part="LED1" gate="G$1" pin="A"/>
+<wire x1="45.72" y1="104.14" x2="45.72" y2="93.98" width="0.1524" layer="91"/>
+<pinref part="U$3" gate="G$1" pin="+IN"/>
+<wire x1="45.72" y1="93.98" x2="45.72" y2="81.28" width="0.1524" layer="91"/>
+<wire x1="58.42" y1="93.98" x2="45.72" y2="93.98" width="0.1524" layer="91"/>
+<junction x="45.72" y="93.98"/>
+</segment>
+</net>
+<net name="N$3" class="0">
+<segment>
+<pinref part="U$3" gate="G$1" pin="-IN"/>
+<pinref part="RP2" gate="G$1" pin="1"/>
+<wire x1="58.42" y1="99.06" x2="55.88" y2="99.06" width="0.1524" layer="91"/>
+<wire x1="55.88" y1="99.06" x2="55.88" y2="83.82" width="0.1524" layer="91"/>
+<pinref part="RP3" gate="G$1" pin="1"/>
+<wire x1="73.66" y1="111.76" x2="55.88" y2="111.76" width="0.1524" layer="91"/>
+<wire x1="55.88" y1="111.76" x2="55.88" y2="99.06" width="0.1524" layer="91"/>
+<junction x="55.88" y="99.06"/>
+</segment>
+</net>
+<net name="N$4" class="0">
+<segment>
+<pinref part="U$3" gate="G$1" pin="OUT"/>
+<wire x1="73.66" y1="96.52" x2="83.82" y2="96.52" width="0.1524" layer="91"/>
+<wire x1="83.82" y1="96.52" x2="83.82" y2="83.82" width="0.1524" layer="91"/>
 <pinref part="U1" gate="G$1" pin="VIN+"/>
-<wire x1="83.82" y1="88.9" x2="83.82" y2="83.82" width="0.1524" layer="91"/>
 <wire x1="83.82" y1="83.82" x2="104.14" y2="83.82" width="0.1524" layer="91"/>
-<wire x1="83.82" y1="88.9" x2="83.82" y2="93.98" width="0.1524" layer="91"/>
-<junction x="83.82" y="88.9"/>
-<pinref part="RP1" gate="G$1" pin="2"/>
-</segment>
-</net>
-<net name="N$1" class="0">
-<segment>
-<pinref part="U1" gate="G$1" pin="VDD"/>
-<wire x1="119.38" y1="91.44" x2="119.38" y2="96.52" width="0.1524" layer="91"/>
-<pinref part="L1" gate="G$1" pin="2"/>
-<pinref part="C2" gate="G$1" pin="2"/>
-<wire x1="119.38" y1="96.52" x2="119.38" y2="99.06" width="0.1524" layer="91"/>
-<wire x1="132.08" y1="101.6" x2="132.08" y2="96.52" width="0.1524" layer="91"/>
-<wire x1="132.08" y1="96.52" x2="119.38" y2="96.52" width="0.1524" layer="91"/>
-<junction x="119.38" y="96.52"/>
-</segment>
-</net>
+<pinref part="RP3" gate="G$1" pin="2"/>
+<wire x1="83.82" y1="111.76" x2="83.82" y2="96.52" width="0.1524" layer="91"/>
+<junction x="83.82" y="96.52"/>
+</segment>
+</net>
